Commit message: add control

File: urdf/mrm.urdf (robot description, URDF)
Before this commit: robot mrm, 6 links, 5 joints
Joints:
- joint base_link_link_01: type prismatic -> revolute
- joint link01_link_02: type revolute -> fixed
- joint link02_link_03: type revolute -> fixed
- joint link03_link_04: type prismatic -> fixed

Commit message: addControl

File: urdf/mrm.urdf (robot description, URDF)
Before this commit: robot mrm, 6 links, 5 joints
Joints:
- joint base_link_link_01: type revolute -> prismatic
- joint link01_link_02: type fixed -> revolute
- joint link02_link_03: type fixed -> revolute
- joint link03_link_04: type fixed -> prismatic

Commit message: AddCamera

File: urdf/mrm.urdf (robot description, URDF)
Before this commit: robot mrm, 6 links, 5 joints
Links:
- added link camera, mass 0.01; collision box size=0.08 0.08 0.08; visual box size=0.08 0.08 0.08
Joints:
- added joint camera_joint: type fixed, parent link_04, child camera, origin xyz=.53 0 0 rpy=0 0 0, axis 0 1 0
- joint link01_link_02: limit lower=-1.04 upper=1.04 effort=1000.0 velocity=0.5 -> lower=-0.35 upper=0.35 effort=1000.0 velocity=0.6
- joint link02_link_03: axis 1 0 0 -> 0 1 0; limit lower=-0.5 upper=0.5 effort=1000.0 velocity=0.5 -> lower=-0.3 upper=0.3 effort=1000.0 velocity=0.6
